File: PlayOnTape Module/PlayOnTape Module.kicad_pcb (KiCad board)
At the start: 2 copper layers, 99.7 x 64.1 mm, 33 parts, among them IC1 0.96_OLED, J1 INPUT, J2 DATASETTE, J3 EXTENSION, J5 PWR, J6 N/C, M1 Mounting, M2 Mounting, M3 Mounting, M4 Mounting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

Commit message: Gerber export
Parts:
- D2: value RECEIVE -> RECORD
- moved U1 6.63 mm to (149.9, 125.7), turned to 0 degrees
- moved G*** 3.81 mm to (120.0, 97.8)
- moved G*** 3.81 mm to (120.7, 97.8)
- moved C1 0.64 mm to (141.6, 94.6)
Connections:
- net RECEIVE renamed RECORD
Routing:
- net SD_SCK: track 0.00 -> 107.8 mm, vias 0 -> 2
- net SD_CS: track 0.00 -> 99.6 mm, vias 0 -> 1
- net CH_Y: track 0.00 -> 90.5 mm, vias 0 -> 2
- net SD_MISO: track 0.00 -> 89.0 mm, vias 0 -> 1
- net BTN_NEXT: track 0.00 -> 85.9 mm, vias 0 -> 1
- net BTN_PLAY: track 0.00 -> 85.1 mm, vias 0 -> 1
- net SD_MOSI: track 0.00 -> 84.1 mm, vias 0 -> 2
- net CH_X: track 0.00 -> 76.3 mm, vias 0 -> 2
- net BTN_STOP: track 0.00 -> 75.1 mm, vias 0 -> 1
- net BTN_PREV: track 0.00 -> 69.6 mm, vias 0 -> 1
- net CH_A: track 0.00 -> 66.4 mm, vias 0 -> 1
- net CH_B: track 0.00 -> 65.5 mm
- net SENSE: track 67.0 -> 103.0 mm
- net OLED_SCL: track 32.5 -> 66.4 mm
- net OLED_SDA: track 34.0 -> 65.2 mm, vias 1 -> 2
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Other:
- board text added: "MOTOR"
- board text added: "PCB Revision A github.com/tebl"
- board text added: "PWR"
- board text added: "READ"
- board text added: "SENSE"
- board text added: "WRITE"

Commit message: Beginning of README
Parts:
- G***: footprint icons:eject -> icons:up

Commit message: Move C1
Parts:
- G***: footprint icons:up -> icons:eject
- moved C1 12.1 mm to (141.0, 106.7), turned to 90 degrees
Routing:
- net +5V: track 196.7 -> 190.7 mm, vias 6 -> 5
- net CH_B: track 65.5 -> 64.4 mm
- net BTN_STOP: track 75.1 -> 74.1 mm
- net /MOTOR: track 67.6 -> 66.8 mm
- net BTN_PLAY: track 85.1 -> 84.5 mm
- net OLED_SCL: track 66.4 -> 67.0 mm
- net OLED_SDA: track 65.2 -> 65.7 mm
Other:
- board text added: "PCB Revision B github.com/tebl"
- board text removed: "PCB Revision A github.com/tebl"
