File: PlayOnTape Module/PlayOnTape Module.kicad_pcb (KiCad board)
At the start: 2 copper layers, 99.7 x 64.1 mm, 33 parts, among them IC1 0.96_OLED, J1 INPUT, J2 DATASETTE, J3 EXTENSION, J5 PWR, J6 N/C, M1 Mounting, M2 Mounting, M3 Mounting, M4 Mounting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

Commit message: Tweak input mounting holes
Parts:
- G***: footprint icons:eject -> icons:next
- G***: footprint icons:eject -> icons:previous
- JP2: value P1_VCC -> P2_VCC
- moved G*** 0.25 mm to (124.5, 139.1), turned to 0 degrees
- moved G*** 0.13 mm to (153.0, 139.1), turned to 0 degrees
Routing:
- net SENSE: track 103.0 -> 103.5 mm

Commit message: Changed to use IDC cable
Parts:
- removed J6: N/C, Pin_Headers:Pin_Header_Straight_1x03_Pitch2.54mm
- J1: footprint PlayOnTape:C64-Cassette-Input -> Connector_IDC:IDC-Header_2x03_P2.54mm_Vertical
- moved J1 49.2 mm to (76.8, 102.9), turned to 180 degrees
- moved C2 4.45 mm to (83.2, 99.1)
- moved U2 4.45 mm to (87.0, 105.4)
Connections:
- D2 pad 1: GND -> RECORD
- R2 pad 2: RECORD -> +5V
Routing:
- net Net-(J1-Pad5): track 70.3 -> 16.7 mm, vias 0 -> 1
- net +5V: track 190.7 -> 218.0 mm, vias 5 -> 3
- net /MOTOR: track 66.8 -> 84.6 mm, vias 3 -> 4
- net SENSE: track 103.5 -> 118.4 mm
- net RECORD: track 18.5 -> 31.6 mm
- net Net-(J1-Pad4): track 44.9 -> 31.8 mm, vias 0 -> 1
- net CH_B: track 64.4 -> 59.9 mm
- net CH_Y: track 90.5 -> 86.1 mm
- net CH_X: track 76.3 -> 71.9 mm
- net CH_A: track 66.4 -> 61.9 mm
- net Net-(J2-Pad4): track 28.9 -> 28.3 mm
Other:
- board text added: "MTR"
- board text added: "RD"
- board text added: "SEN"
- board text added: "WR"
- board text removed: "MOTOR"
- board text removed: "READ"
- board text removed: "SENSE"
- board text removed: "WRITE"

Commit message: Silkscreen tweaks
Other:
- board text added: "JP1/JP2: Link 1-2 when OLED pin 1 is GND, 2-3 if VCC"
